File: D97cpu.kicad_sch (KiCad schematic)
At the start: 31 parts, among them IC2 NCP730BMT330TBG, J3 Conn_01x01, Q1 PMZB200UNEYL, Q1A1 BC857BDW1, Q1B1 BC857BDW1, Q2 PMZB200UNEYL, Q2A1 BC847BDW1, Q2B1 BC847BDW1, Q4 PMZB200UNEYL, Q5 PMZB200UNEYL, U1 AVR-64DA32

Commit message: initial commit
Other:
- title: RTB D98 Function Decoder -> RTB D97 FN Decoder Toolkit
Changed lines of the file:
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@@
 	(paper "A4")
 	(title_block
-		(title "RTB D98 Function Decoder")
-		(date "2025-11-18")
+		(title "RTB D97 FN Decoder Toolkit")
+		(date "2025-11-22")
 		(rev "0")
 		(company "Frank Schumacher")
 		(comment 1 "'naked' DCC decoder project")
-		(comment 2 "D98.0")
+		(comment 2 "D97.0")
 		(comment 4 "Licensed under the Apache License, Version 2")
 	)
@@
 		)
 		(instances
-			(project "D98"
+			(project "D97"
 				(path "/770f17cd-ae87-4649-af39-9a95ef9cf5c7/00000000-0000-0000-0000-00005b6c6b9d"
 					(reference "U1")
@@
 		)
 		(instances
-			(project "D98"
+			(project "D97"
 				(path "/770f17cd-ae87-4649-af39-9a95ef9cf5c7/00000000-0000-0000-0000-00005b6c6b9d"
 					(reference "#PWR0110")
@@
 		)
 		(instances
-			(project "D98"
+			(project "D97"
 				(path "/770f17cd-ae87-4649-af39-9a95ef9cf5c7/00000000-0000-0000-0000-00005b6c6b9d"
 					(reference "C7")
@@
 		)
 		(instances
-			(project "D98"
+			(project "D97"
 				(path "/770f17cd-ae87-4649-af39-9a95ef9cf5c7/00000000-0000-0000-0000-00005b6c6b9d"
 					(reference "IC2")
@@
 		)
 		(instances
-			(project "D98"
+			(project "D97"
 				(path "/770f17cd-ae87-4649-af39-9a95ef9cf5c7/00000000-0000-0000-0000-00005b6c6b9d"
 					(reference "R20")
@@
 		)
 		(instances
-			(project "D98"
+			(project "D97"
 				(path "/770f17cd-ae87-4649-af39-9a95ef9cf5c7/00000000-0000-0000-0000-00005b6c6b9d"
 					(reference "R19")
@@
 		)
 		(instances
-			(project "D98"
+			(project "D97"
 				(path "/770f17cd-ae87-4649-af39-9a95ef9cf5c7/00000000-0000-0000-0000-00005b6c6b9d"
 					(reference "C3")
@@
 		)
 		(instances
-			(project "D98"
+			(project "D97"
 				(path "/770f17cd-ae87-4649-af39-9a95ef9cf5c7/00000000-0000-0000-0000-00005b6c6b9d"
 					(reference "D3")
@@
 		)
 		(instances
-			(project "D98"
+			(project "D97"
 				(path "/770f17cd-ae87-4649-af39-9a95ef9cf5c7/00000000-0000-0000-0000-00005b6c6b9d"
 					(reference "#PWR030")
@@
 		)
 		(instances
-			(project "D98"
+			(project "D97"
 				(path "/770f17cd-ae87-4649-af39-9a95ef9cf5c7/00000000-0000-0000-0000-00005b6c6b9d"
 					(reference "R9")
@@
 		)
 		(instances
-			(project "D98"
+			(project "D97"
 				(path "/770f17cd-ae87-4649-af39-9a95ef9cf5c7/00000000-0000-0000-0000-00005b6c6b9d"
 					(reference "#PWR016")
@@
 		)
 		(instances
-			(project "D98"
+			(project "D97"
 				(path "/770f17cd-ae87-4649-af39-9a95ef9cf5c7/00000000-0000-0000-0000-00005b6c6b9d"
 					(reference "#PWR017")
@@
 		)
 		(instances
-			(project "D98"
+			(project "D97"
 				(path "/770f17cd-ae87-4649-af39-9a95ef9cf5c7/00000000-0000-0000-0000-00005b6c6b9d"
 					(reference "#PWR018")
@@
 		)
 		(instances
-			(project "D98"
+			(project "D97"
 				(path "/770f17cd-ae87-4649-af39-9a95ef9cf5c7/00000000-0000-0000-0000-00005b6c6b9d"
 					(reference "#PWR032")
@@
 		)
 		(instances
-			(project "D98"
+			(project "D97"
 				(path "/770f17cd-ae87-4649-af39-9a95ef9cf5c7/00000000-0000-0000-0000-00005b6c6b9d"
 					(reference "#PWR019")
@@
 		)
 		(instances
-			(project "D98"
+			(project "D97"
 				(path "/770f17cd-ae87-4649-af39-9a95ef9cf5c7/00000000-0000-0000-0000-00005b6c6b9d"
 					(reference "R17")
@@
 		)
 		(instances
-			(project "D98"
+			(project "D97"
 				(path "/770f17cd-ae87-4649-af39-9a95ef9cf5c7/00000000-0000-0000-0000-00005b6c6b9d"
 					(reference "Q2B1")
@@
 		)
 		(instances
-			(project "D98"
+			(project "D97"
 				(path "/770f17cd-ae87-4649-af39-9a95ef9cf5c7/00000000-0000-0000-0000-00005b6c6b9d"
 					(reference "#PWR029")
@@
 		)
 		(instances
-			(project "D98"
+			(project "D97"
 				(path "/770f17cd-ae87-4649-af39-9a95ef9cf5c7/00000000-0000-0000-0000-00005b6c6b9d"
 					(reference "#PWR012")
@@
 		)
 		(instances
-			(project ""
+			(project "D97"
 				(path "/770f17cd-ae87-4649-af39-9a95ef9cf5c7/00000000-0000-0000-0000-00005b6c6b9d"
 					(reference "#PWR01")
@@
 		)
 		(instances
-			(project "D98"
+			(project "D97"
 				(path "/770f17cd-ae87-4649-af39-9a95ef9cf5c7/00000000-0000-0000-0000-00005b6c6b9d"
 					(reference "R1")
@@
 		)
 		(instances
-			(project "D98"
+			(project "D97"
 				(path "/770f17cd-ae87-4649-af39-9a95ef9cf5c7/00000000-0000-0000-0000-00005b6c6b9d"
 					(reference "R3")
@@
 		)
 		(instances
-			(project ""
+			(project "D97"
 				(path "/770f17cd-ae87-4649-af39-9a95ef9cf5c7/00000000-0000-0000-0000-00005b6c6b9d"
 					(reference "#PWR020")
@@
 		)
 		(instances
-			(project "D98"
+			(project "D97"
 				(path "/770f17cd-ae87-4649-af39-9a95ef9cf5c7/00000000-0000-0000-0000-00005b6c6b9d"
 					(reference "#PWR011")
@@
 		)
 		(instances
-			(project "D98"
+			(project "D97"
 				(path "/770f17cd-ae87-4649-af39-9a95ef9cf5c7/00000000-0000-0000-0000-00005b6c6b9d"
 					(reference "Q1A1")
@@
 		)
 		(instances
-			(project "D98"
+			(project "D97"
 				(path "/770f17cd-ae87-4649-af39-9a95ef9cf5c7/00000000-0000-0000-0000-00005b6c6b9d"
 					(reference "R13")
@@
 		)
 		(instances
-			(project ""
+			(project "D97"
 				(path "/770f17cd-ae87-4649-af39-9a95ef9cf5c7/00000000-0000-0000-0000-00005b6c6b9d"
 					(reference "Q1")
@@
 		)
 		(instances
-			(project "D98"
+			(project "D97"
 				(path "/770f17cd-ae87-4649-af39-9a95ef9cf5c7/00000000-0000-0000-0000-00005b6c6b9d"
 					(reference "D6")
@@
 		)
 		(instances
-			(project "D98"
+			(project "D97"
 				(path "/770f17cd-ae87-4649-af39-9a95ef9cf5c7/00000000-0000-0000-0000-00005b6c6b9d"
 					(reference "R14")
@@
 		)
 		(instances
-			(project "D98"
+			(project "D97"
 				(path "/770f17cd-ae87-4649-af39-9a95ef9cf5c7/00000000-0000-0000-0000-00005b6c6b9d"
 					(reference "Q4")
@@
 		)
 		(instances
-			(project ""
+			(project "D97"
 				(path "/770f17cd-ae87-4649-af39-9a95ef9cf5c7/00000000-0000-0000-0000-00005b6c6b9d"
 					(reference "J3")
@@
 		)
 		(instances
-			(project "D98"
+			(project "D97"
 				(path "/770f17cd-ae87-4649-af39-9a95ef9cf5c7/00000000-0000-0000-0000-00005b6c6b9d"
 					(reference "R6")
@@
 		)
 		(instances
-			(project ""
+			(project "D97"
 				(path "/770f17cd-ae87-4649-af39-9a95ef9cf5c7/00000000-0000-0000-0000-00005b6c6b9d"
 					(reference "D1")
@@
 		)
 		(instances
-			(project "D98"
+			(project "D97"
 				(path "/770f17cd-ae87-4649-af39-9a95ef9cf5c7/00000000-0000-0000-0000-00005b6c6b9d"
 					(reference "Q5")
@@
 		)
 		(instances
-			(project "D98"
+			(project "D97"
 				(path "/770f17cd-ae87-4649-af39-9a95ef9cf5c7/00000000-0000-0000-0000-00005b6c6b9d"
 					(reference "#PWR031")
@@
 		)
 		(instances
-			(project "D98"
+			(project "D97"
 				(path "/770f17cd-ae87-4649-af39-9a95ef9cf5c7/00000000-0000-0000-0000-00005b6c6b9d"
 					(reference "Q2")
@@
 		)
 		(instances
-			(project "D98"
+			(project "D97"
 				(path "/770f17cd-ae87-4649-af39-9a95ef9cf5c7/00000000-0000-0000-0000-00005b6c6b9d"
 					(reference "D5")
@@
 		)
 		(instances
-			(project "D98"
+			(project "D97"
 				(path "/770f17cd-ae87-4649-af39-9a95ef9cf5c7/00000000-0000-0000-0000-00005b6c6b9d"
 					(reference "#PWR010")
@@
 		)
 		(instances
-			(project "D98"
+			(project "D97"
 				(path "/770f17cd-ae87-4649-af39-9a95ef9cf5c7/00000000-0000-0000-0000-00005b6c6b9d"
 					(reference "#PWR013")
@@
 		)
 		(instances
-			(project "D98"
+			(project "D97"
 				(path "/770f17cd-ae87-4649-af39-9a95ef9cf5c7/00000000-0000-0000-0000-00005b6c6b9d"
 					(reference "Q2A1")
@@
 		)
 		(instances
-			(project "D98"
+			(project "D97"
 				(path "/770f17cd-ae87-4649-af39-9a95ef9cf5c7/00000000-0000-0000-0000-00005b6c6b9d"
 					(reference "R5")
@@
 		)
 		(instances
-			(project "D98"
+			(project "D97"
 				(path "/770f17cd-ae87-4649-af39-9a95ef9cf5c7/00000000-0000-0000-0000-00005b6c6b9d"
 					(reference "#PWR06")
@@
 		)
 		(instances
-			(project "D98"
+			(project "D97"
 				(path "/770f17cd-ae87-4649-af39-9a95ef9cf5c7/00000000-0000-0000-0000-00005b6c6b9d"
 					(reference "R4")
@@
 		)
 		(instances
-			(project "D98"
+			(project "D97"
 				(path "/770f17cd-ae87-4649-af39-9a95ef9cf5c7/00000000-0000-0000-0000-00005b6c6b9d"
 					(reference "D7")
@@
 		)
 		(instances
-			(project "D98"
+			(project "D97"
 				(path "/770f17cd-ae87-4649-af39-9a95ef9cf5c7/00000000-0000-0000-0000-00005b6c6b9d"
 					(reference "Q1B1")
@@
 		)
 		(instances
-			(project "D98"
+			(project "D97"
 				(path "/770f17cd-ae87-4649-af39-9a95ef9cf5c7/00000000-0000-0000-0000-00005b6c6b9d"
 					(reference "R16")
@@
 		)
 		(instances
-			(project "D98"
+			(project "D97"
 				(path "/770f17cd-ae87-4649-af39-9a95ef9cf5c7/00000000-0000-0000-0000-00005b6c6b9d"
 					(reference "R15")
@@
 		)
 		(instances
-			(project "D98"
+			(project "D97"
 				(path "/770f17cd-ae87-4649-af39-9a95ef9cf5c7/00000000-0000-0000-0000-00005b6c6b9d"
 					(reference "#PWR014")
