File: D97prt.kicad_sch (KiCad schematic)
At the start: 6 parts, among them IC1 74HC595BQ,115, IC3 74HC595BQ,115, IC4 74HC595BQ,115, IC5 74HC595BQ,115, U4 WS2812-2020, U5 WS2812-2020

Commit message: initial commit
Other:
- title: RTB D98 Function Decoder -> RTB D97 FN Decoder Toolkit
Changed lines of the file:
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@@
 	(paper "A4")
 	(title_block
-		(title "RTB D98 Function Decoder")
-		(date "2025-11-18")
+		(title "RTB D97 FN Decoder Toolkit")
+		(date "2025-11-22")
 		(rev "0")
 		(company "Frank Schumacher")
 		(comment 1 "'naked' DCC decoder project")
-		(comment 2 "D98.0")
+		(comment 2 "D97.0")
 		(comment 4 "Licensed under the Apache License, Version 2")
 	)
@@
 		)
 		(instances
-			(project "D98"
+			(project "D97"
 				(path "/770f17cd-ae87-4649-af39-9a95ef9cf5c7/00000000-0000-0000-0000-00005ca7768a"
 					(reference "#PWR015")
@@
 		)
 		(instances
-			(project "D98"
+			(project "D97"
 				(path "/770f17cd-ae87-4649-af39-9a95ef9cf5c7/00000000-0000-0000-0000-00005ca7768a"
 					(reference "IC1")
@@
 		)
 		(instances
-			(project "D98"
+			(project "D97"
 				(path "/770f17cd-ae87-4649-af39-9a95ef9cf5c7/00000000-0000-0000-0000-00005ca7768a"
 					(reference "#PWR022")
@@
 		)
 		(instances
-			(project "D98"
+			(project "D97"
 				(path "/770f17cd-ae87-4649-af39-9a95ef9cf5c7/00000000-0000-0000-0000-00005ca7768a"
 					(reference "#PWR028")
@@
 		)
 		(instances
-			(project "D98"
+			(project "D97"
 				(path "/770f17cd-ae87-4649-af39-9a95ef9cf5c7/00000000-0000-0000-0000-00005ca7768a"
 					(reference "IC5")
@@
 		)
 		(instances
-			(project "D98"
+			(project "D97"
 				(path "/770f17cd-ae87-4649-af39-9a95ef9cf5c7/00000000-0000-0000-0000-00005ca7768a"
 					(reference "#PWR08")
@@
 		)
 		(instances
-			(project "D98"
+			(project "D97"
 				(path "/770f17cd-ae87-4649-af39-9a95ef9cf5c7/00000000-0000-0000-0000-00005ca7768a"
 					(reference "#PWR024")
@@
 		)
 		(instances
-			(project "D98"
+			(project "D97"
 				(path "/770f17cd-ae87-4649-af39-9a95ef9cf5c7/00000000-0000-0000-0000-00005ca7768a"
 					(reference "#PWR025")
@@
 		)
 		(instances
-			(project "D98"
+			(project "D97"
 				(path "/770f17cd-ae87-4649-af39-9a95ef9cf5c7/00000000-0000-0000-0000-00005ca7768a"
 					(reference "U5")
@@
 		)
 		(instances
-			(project "D98"
+			(project "D97"
 				(path "/770f17cd-ae87-4649-af39-9a95ef9cf5c7/00000000-0000-0000-0000-00005ca7768a"
 					(reference "#PWR021")
@@
 		)
 		(instances
-			(project "D98"
+			(project "D97"
 				(path "/770f17cd-ae87-4649-af39-9a95ef9cf5c7/00000000-0000-0000-0000-00005ca7768a"
 					(reference "#PWR09")
@@
 		)
 		(instances
-			(project "D98"
+			(project "D97"
 				(path "/770f17cd-ae87-4649-af39-9a95ef9cf5c7/00000000-0000-0000-0000-00005ca7768a"
 					(reference "#PWR023")
@@
 		)
 		(instances
-			(project "D98"
+			(project "D97"
 				(path "/770f17cd-ae87-4649-af39-9a95ef9cf5c7/00000000-0000-0000-0000-00005ca7768a"
 					(reference "#PWR027")
@@
 		)
 		(instances
-			(project "D98"
+			(project "D97"
 				(path "/770f17cd-ae87-4649-af39-9a95ef9cf5c7/00000000-0000-0000-0000-00005ca7768a"
 					(reference "IC3")
@@
 		)
 		(instances
-			(project "D98"
+			(project "D97"
 				(path "/770f17cd-ae87-4649-af39-9a95ef9cf5c7/00000000-0000-0000-0000-00005ca7768a"
 					(reference "U4")
@@
 		)
 		(instances
-			(project "D98"
+			(project "D97"
 				(path "/770f17cd-ae87-4649-af39-9a95ef9cf5c7/00000000-0000-0000-0000-00005ca7768a"
 					(reference "IC4")
@@
 		)
 		(instances
-			(project "D98"
+			(project "D97"
 				(path "/770f17cd-ae87-4649-af39-9a95ef9cf5c7/00000000-0000-0000-0000-00005ca7768a"
 					(reference "#PWR026")
@@
 		)
 		(instances
-			(project "D98"
+			(project "D97"
 				(path "/770f17cd-ae87-4649-af39-9a95ef9cf5c7/00000000-0000-0000-0000-00005ca7768a"
 					(reference "#PWR07")
