File: D97ex3.kicad_sch (KiCad schematic)
At the start: 31 parts, among them IC2 NCP730BMT330TBG, J3 Conn_01x01, Q1 PMZB200UNEYL, Q1A1 BC857BDW1, Q1B1 BC857BDW1, Q2 PMZB200UNEYL, Q2A1 BC847BDW1, Q2B1 BC847BDW1, Q4 PMZB200UNEYL, Q5 PMZB200UNEYL, U1 AVR-64DA32

Commit message: initial commit
Parts:
- removed D5: LED, LED_SMD:LED_0402_1005Metric, symbol Device:LED
- removed J3: Conn_01x01, TestPoint:TestPoint_Pad_D1.0mm, symbol Connector_Generic:Conn_01x01
- removed Q1, Q2, Q5: PMZB200UNEYL, PMZB200UNEYL, symbol RTB:PMZB200UNEYL
- removed R1: 3.3k, Resistor_SMD:R_0402_1005Metric, symbol Device:R
Connections:
- net AUX1: no longer names the net of U1.32 (PA2)
- net AUX2: no longer names the net of U1.1 (PA3)
- net AUX3: no longer names the net of U1.2 (PA4)
- net AUX4: no longer names the net of U1.3 (PA5)
- net AUX5: no longer names the net of U1.4 (PA6)
- net AUX6: no longer names the net of U1.5 (PA7)
- net AUX7: no longer names the net of U1.8 (PC2)
- net AUX8: no longer names the net of U1.9 (PC3)
- net CAP_ena: no longer names the net of U1.17 (PD7)
- net DAC_out: no longer names the net of U1.16 (PD6)
- net F0f: no longer names the net of U1.31 (PA1)
- net F0r: no longer names the net of U1.30 (EXTCLK/PA0)
- net IN1: no longer names the net of U1.13 (PD3)
- net IN2: no longer names the net of U1.14 (PD4)
- net LED.hbt: no longer names the net of U1.25 (PF5)
- net SERVO_dat: no longer names the net of U1.20 (PF0/TOSC1)
- net SERVO_pwr: no longer names the net of U1.21 (PF1/TOSC2)
- net SUSI_scl: no longer names the net of U1.23 (PF3)
- net SUSI_sda: no longer names the net of U1.22 (PF2)
- net WS28xx: no longer names the net of U1.6 (PC0)
- net iAUX: no longer names the net of U1.12 (PD2)
Other:
- note added: "- can read/write CVs on Programming Track - Railcom (Pom, xPom, DCC-A, DCC-R, FW-update)"
- note added: "Proper DCC Decoder"
- note removed: "..."
- note removed: "FL/AUX Ports"
- note removed: "Heartbeat LED"
- note removed: "Test Point"
- note removed: "UPDI"
