File: D97ex3.kicad_sch (KiCad schematic)
At the start: 25 parts, among them IC2 NCP730BMT330TBG, Q1A1 BC857BDW1, Q1B1 BC857BDW1, Q2A1 BC847BDW1, Q2B1 BC847BDW1, Q4 PMZB200UNEYL, U1 AVR-64DA32

Commit message: initial commit
Other:
- note added: "Example 3"
- note removed: "Proper DCC Decoder"
Changed lines of the file:
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@@
 		(comment 1 "'naked' DCC decoder project")
 		(comment 2 "D97.0")
+		(comment 3 "Example 3: DCC Decoder /w Railcom")
 		(comment 4 "Licensed under the Apache License, Version 2")
 	)
@@
 	(text "- can read/write CVs on Programming Track\n- Railcom (Pom, xPom, DCC-A, DCC-R, FW-update)"
 		(exclude_from_sim no)
-		(at 140.716 91.44 0)
+		(at 140.716 90.17 0)
 		(effects
 			(font
@@
 		)
 	)
-	(text "Proper DCC Decoder"
+	(text "Example 3"
 		(exclude_from_sim no)
 		(at 140.462 80.772 0)
