File: D97.kicad_sch (KiCad schematic)
At the start: 0 parts

Commit message: initial commit
Other:
- sheet CPU: file D98cpu.kicad_sch -> D97cpu.kicad_sch
- sheet External Ports: file D98prt.kicad_sch -> D97prt.kicad_sch
- title: RTB D98 Function Decoder -> RTB D97 FN Decoder Toolkit
Changed lines of the file:
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@@
 	(paper "A4")
 	(title_block
-		(title "RTB D98 Function Decoder")
-		(date "2025-11-18")
+		(title "RTB D97 FN Decoder Toolkit")
+		(date "2025-11-22")
 		(rev "0")
 		(company "Frank Schumacher")
 		(comment 1 "'naked' DCC decoder project")
-		(comment 2 "D98.0")
+		(comment 2 "D97.0")
 		(comment 4 "Licensed under the Apache License, Version 2")
 	)
@@
 			)
 		)
-		(property "Sheetfile" "D98cpu.kicad_sch"
+		(property "Sheetfile" "D97cpu.kicad_sch"
 			(at 96.52 102.4792 0)
 			(effects
@@
 		)
 		(instances
-			(project "D98"
+			(project "D97"
 				(path "/770f17cd-ae87-4649-af39-9a95ef9cf5c7"
 					(page "2")
@@
 			)
 		)
-		(property "Sheetfile" "D98prt.kicad_sch"
+		(property "Sheetfile" "D97prt.kicad_sch"
 			(at 157.48 102.4792 0)
 			(effects
@@
 		)
 		(instances
-			(project "D98"
+			(project "D97"
 				(path "/770f17cd-ae87-4649-af39-9a95ef9cf5c7"
 					(page "4")

Commit message: initial commit
Other:
- added sheet Example 1 (D97ex1.kicad_sch)
- added sheet Example 2 (D97ex2.kicad_sch)
- added sheet Example 3 (D97ex3.kicad_sch)
- note added: "DCC decoder /w CV reading on ProgTrack /w Railcom"
- note added: "Most simplistic DCC decoder"
- note added: "Simplistic DCC decoder /w CV reading on ProgTrack"
Changed lines of the file:
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@@
 		(comment 4 "Licensed under the Apache License, Version 2")
 	)
-	(sheet
-		(at 96.52 82.55)
+	(text "DCC decoder\n/w CV reading on ProgTrack\n/w Railcom"
+		(exclude_from_sim no)
+		(at 42.926 95.25 0)
+		(effects
+			(font
+				(size 1.27 1.27)
+			)
+		)
+	)
+	(text "Simplistic DCC decoder\n/w CV reading on ProgTrack"
+		(exclude_from_sim no)
+		(at 43.18 62.484 0)
+		(effects
+			(font
+				(size 1.27 1.27)
+			)
+		)
+	)
+	(text "Most simplistic DCC decoder"
+		(exclude_from_sim no)
+		(at 44.958 32.766 0)
+		(effects
+			(font
+				(size 1.27 1.27)
+			)
+		)
+	)
+	(sheet
+		(at 158.75 86.36)
 		(size 44.45 19.05)
 		(exclude_from_sim no)
@@
 		)
 		(property "Sheetname" "CPU"
-			(at 96.52 81.4701 0)
+			(at 158.75 85.2801 0)
 			(effects
 				(font
@@
 		)
 		(property "Sheetfile" "D97cpu.kicad_sch"
-			(at 96.52 102.4792 0)
+			(at 158.75 106.2892 0)
 			(effects
 				(font
@@
 	)
 	(sheet
-		(at 157.48 82.55)
+		(at 219.71 86.36)
 		(size 50.8 19.05)
 		(exclude_from_sim no)
@@
 		)
 		(property "Sheetname" "External Ports"
-			(at 157.48 81.4701 0)
+			(at 219.71 85.2801 0)
 			(effects
 				(font
@@
 		)
 		(property "Sheetfile" "D97prt.kicad_sch"
-			(at 157.48 102.4792 0)
+			(at 219.71 106.2892 0)
 			(effects
 				(font
@@
 				)
 			)
+		)
+	)
+	(sheet
+		(at 22.225 85.725)
+		(size 44.45 19.05)
+		(exclude_from_sim no)
+		(in_bom yes)
+		(on_board yes)
+		(dnp no)
+		(fields_autoplaced yes)
+		(stroke
+			(width 0)
+			(type solid)
+		)
+		(fill
+			(color 0 0 0 0.0000)
+		)
+		(property "Sheetname" "Example 3"
+			(at 22.225 84.6451 0)
+			(effects
+				(font
+					(size 2.0066 2.0066)
+				)
+				(justify left bottom)
+			)
+		)
+		(property "Sheetfile" "D97ex3.kicad_sch"
+			(at 22.225 105.6542 0)
+			(effects
+				(font
+					(size 2.0066 2.0066)
+				)
+				(justify left top)
+			)
+		)
+		(instances
+			(project "D97"
+				(path "/770f17cd-ae87-4649-af39-9a95ef9cf5c7"
+					(page "6")
+				)
+			)
+		)
+	)
+	(sheet
+		(at 22.225 52.705)
+		(size 44.45 19.05)
+		(exclude_from_sim no)
+		(in_bom yes)
+		(on_board yes)
+		(dnp no)
+		(fields_autoplaced yes)
+		(stroke
+			(width 0)
+			(type solid)
+		)
+		(fill
+			(color 0 0 0 0.0000)
+		)
+		(property "Sheetname" "Example 2"
+			(at 22.225 51.6251 0)
+			(effects
+				(font
+					(size 2.0066 2.0066)
+				)
+				(justify left bottom)
+			)
+		)
+		(property "Sheetfile" "D97ex2.kicad_sch"
+			(at 22.225 72.6342 0)
+			(effects
+				(font
+					(size 2.0066 2.0066)
+				)
+				(justify left top)
+			)
+		)
+		(instances
+			(project "D97"
+				(path "/770f17cd-ae87-4649-af39-9a95ef9cf5c7"
+					(page "5")
+				)
+			)
+		)
+	)
+	(sheet
+		(at 21.59 22.86)
+		(size 44.45 19.05)
+		(exclude_from_sim no)
+		(in_bom yes)
+		(on_board yes)
+		(dnp no)
+		(fields_autoplaced yes)
+		(stroke
+			(width 0)
+			(type solid)
+		)
+		(fill
+			(color 0 0 0 0.0000)
+		)
+		(property "Sheetname" "Example 1"
+			(at 21.59 21.7801 0)
+			(effects
+				(font
+					(size 2.0066 2.0066)
+				)
+				(justify left bottom)
+			)
+		)
+		(property "Sheetfile" "D97ex1.kicad_sch"
+			(at 21.59 42.7892 0)
+			(effects
+				(font
+					(size 2.0066 2.0066)
+				)
+				(justify left top)
+			)
+		)
+		(instances
+			(project "D97"
+				(path "/770f17cd-ae87-4649-af39-9a95ef9cf5c7"
+					(page "3")
+				)
+			)

Commit message: initial commit
Other:
- added sheet Example 4 (D97ex4.kicad_sch)
Changed lines of the file:
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@@
+		)
+	)
+	(sheet
+		(at 22.86 119.38)
+		(size 44.45 19.05)
+		(exclude_from_sim no)
+		(in_bom yes)
+		(on_board yes)
+		(dnp no)
+		(fields_autoplaced yes)
+		(stroke
+			(width 0)
+			(type solid)
+		)
+		(fill
+			(color 0 0 0 0.0000)
+		)
+		(property "Sheetname" "Example 4"
+			(at 22.86 118.3001 0)
+			(effects
+				(font
+					(size 2.0066 2.0066)
+				)
+				(justify left bottom)
+			)
+		)
+		(property "Sheetfile" "D97ex4.kicad_sch"
+			(at 22.86 139.3092 0)
+			(effects
+				(font
+					(size 2.0066 2.0066)
+				)
+				(justify left top)
+			)
+		)
+		(instances
+			(project "D97"
+				(path "/770f17cd-ae87-4649-af39-9a95ef9cf5c7"
+					(page "7")
+				)
+			)
 		)
 	)

Commit message: initial commit
Other:
- note added: "Simple DCC decoder /w CV reading on ProgTrack"
- note added: "Simplistic DCC decoder /w CV reading on ProgTrack /w WS28xx neo pixel"
- note added: "Very simple DCC decoder"
- note removed: "Most simplistic DCC decoder"
- note removed: "Simplistic DCC decoder /w CV reading on ProgTrack"
Changed lines of the file:
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@@
 	(text "DCC decoder\n/w CV reading on ProgTrack\n/w Railcom"
 		(exclude_from_sim no)
-		(at 42.926 95.25 0)
+		(at 30.734 94.488 0)
 		(effects
 			(font
 				(size 1.27 1.27)
 			)
+			(justify left)
 		)
 	)
-	(text "Simplistic DCC decoder\n/w CV reading on ProgTrack"
+	(text "Simple DCC decoder\n/w CV reading on ProgTrack"
 		(exclude_from_sim no)
-		(at 43.18 62.484 0)
+		(at 31.242 61.976 0)
 		(effects
 			(font
 				(size 1.27 1.27)
 			)
+			(justify left)
 		)
 	)
-	(text "Most simplistic DCC decoder"
+	(text "Very simple DCC decoder"
 		(exclude_from_sim no)
-		(at 44.958 32.766 0)
+		(at 31.242 32.258 0)
 		(effects
 			(font
 				(size 1.27 1.27)
 			)
+			(justify left)
 		)
 	)
+	(text "Simplistic DCC decoder\n/w CV reading on ProgTrack\n/w WS28xx neo pixel"
+		(exclude_from_sim no)
+		(at 30.734 129.286 0)
+		(effects
+			(font
+				(size 1.27 1.27)
+			)
+			(justify left)
+		)
+	)
