File: D97ex1.kicad_sch (KiCad schematic)
At the start: 12 parts, among them IC2 NCP730BMT330TBG, U1 AVR-64DA32

Commit message: initial commit
Other:
- note added: "- can only write CVs (no reading)"
- note added: "Example 1"
- note removed: "- can only write CVs on Programming Track"
- note removed: "Very simple DCC Decoder"
Changed lines of the file:
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@@
 		(comment 1 "'naked' DCC decoder project")
 		(comment 2 "D97.0")
-		(comment 3 "Example 1: Simple DCC decoder")
+		(comment 3 "Example 1: Very simple DCC decoder")
 		(comment 4 "Licensed under the Apache License, Version 2")
 	)
@@
 		)
 	)
-	(text "- can only write CVs on Programming Track"
+	(text "- can only write CVs (no reading)"
 		(exclude_from_sim no)
 		(at 138.684 92.202 0)
@@
 		)
 	)
-	(text "Very simple DCC Decoder"
+	(text "Example 1"
 		(exclude_from_sim no)
 		(at 137.668 84.836 0)
