File: D97ex2.kicad_sch (KiCad schematic)
At the start: 14 parts, among them IC2 NCP730BMT330TBG, Q4 PMZB200UNEYL, U1 AVR-64DA32

Commit message: initial commit
Other:
- note added: "Example 2"
- note removed: "Simple DCC Decoder"
Changed lines of the file:
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@@
 		)
 	)
-	(text "Simple DCC Decoder"
+	(text "Example 2"
 		(exclude_from_sim no)
 		(at 137.668 83.82 0)
