File: D97ex4.kicad_sch (KiCad schematic)
At the start: 25 parts, among them IC2 NCP730BMT330TBG, Q1A1 BC857BDW1, Q1B1 BC857BDW1, Q2A1 BC847BDW1, Q2B1 BC847BDW1, Q4 PMZB200UNEYL, U1 AVR-64DA32

Commit message: initial commit
Parts:
- removed Q1A1, Q1B1: BC857BDW1, Package_TO_SOT_SMD:SOT-666, symbol Transistor_BJT:BC857BDW1
- removed Q2A1, Q2B1: BC847BDW1, Package_TO_SOT_SMD:SOT-666, symbol Transistor_BJT:BC847BDW1
- removed R14, R9: 220k, Resistor_SMD:R_0402_1005Metric, symbol Device:R
- removed R16, R17: 9.1k, Resistor_SMD:R_0402_1005Metric, symbol Device:R
- removed R4: 22, Resistor_SMD:R_0402_1005Metric, symbol Device:R
- removed R5, R6: 10k, Resistor_SMD:R_0402_1005Metric, symbol Device:R
- added U2, U3: WS2812-2020, RTB:WS2812-2020, symbol RTB:WS2812-2020
Connections:
- net GNDD: now also U2.2 (GND), U3.2 (GND)
- net VDD: now also U2.4 (VDD), U3.4 (VDD)
- net WS28xx: now reaches U1.6 (PC0)
- net WS28xx: now also U2.3 (DI)
- no-connect marks 3 -> 4
Other:
- note added: "- can read/write CVs on Programming Track - connects to WS28xx Neo Pixel LEDs"
- note added: "DCC Decoder /w WS28xx LEDs"
- note added: "WS: Neo Pixel"
- note added: "up to 32 single color LEDs or 10 RGB LEDs"
- note removed: "- can read/write CVs on Programming Track - Railcom (Pom, xPom, DCC-A, DCC-R, FW-update)"
- note removed: "DCC voltage measure"
- note removed: "Proper DCC Decoder"
- note removed: "Railcom TX"
- note removed: "VDD=5V: 33 Ohm"
- note removed: "Voltage Divider"

Commit message: initial commit
Other:
- note added: "- can read/write CVs on Programming Track - driving WS28xx Neo Pixel LEDs"
- note added: "Example 4"
- note removed: "- can read/write CVs on Programming Track - connects to WS28xx Neo Pixel LEDs"
- note removed: "DCC Decoder /w WS28xx LEDs"
Changed lines of the file:
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@@
 		(comment 1 "'naked' DCC decoder project")
 		(comment 2 "D97.0")
+		(comment 3 "Example 4: Simple DCC Decoder /w WS28xx NeoPixel")
 		(comment 4 "Licensed under the Apache License, Version 2")
 	)
@@
 		)
 	)
-	(text "- can read/write CVs on Programming Track\n- connects to WS28xx Neo Pixel LEDs"
-		(exclude_from_sim no)
-		(at 140.716 91.44 0)
+	(text "- can read/write CVs on Programming Track\n- driving WS28xx Neo Pixel LEDs"
+		(exclude_from_sim no)
+		(at 140.716 90.17 0)
 		(effects
 			(font
@@
 		)
 	)
-	(text "DCC Decoder /w WS28xx LEDs"
+	(text "Example 4"
 		(exclude_from_sim no)
 		(at 140.462 80.772 0)
@@
 	(polyline
 		(pts
-			(xy 269.24 161.29) (xy 81.915 161.29)
+			(xy 277.495 161.29) (xy 81.915 161.29)
 		)
 		(stroke
@@
 	(polyline
 		(pts
-			(xy 269.24 114.935) (xy 269.24 161.29)
+			(xy 277.495 114.935) (xy 277.495 161.29)
 		)
 		(stroke
@@
 	(polyline
 		(pts
-			(xy 81.915 114.935) (xy 269.875 114.935)
-		)
-		(stroke
+			(xy 81.915 114.935) (xy 277.495 114.935)
+		)
+		(stroke
